File: Aqua.kicad_pcb (KiCad board)
At the start: 2 copper layers, 160 x 102.9 mm, 18 parts, among them J1 Screw_Terminal_01x02, J2 Screw_Terminal_01x02, J3 Screw_Terminal_01x02, J4 Screw_Terminal_01x02, J5 Screw_Terminal_01x02, J6 Screw_Terminal_01x02, J7 USB_B_Micro, U1 NodeMCU_1.0_(ESP-12E), U2 74HC595, U3 74HC595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

Commit message: WIP
Parts:
- added C1: 0.1mF, Capacitor_THT:CP_Radial_D7.5mm_P2.50mm, F.Cu at (152.4, 29.2)
- added C2: 0.1mF, Capacitor_THT:CP_Radial_D7.5mm_P2.50mm, F.Cu at (149.9, 64.8)
- added C3: 0.1mF, Capacitor_THT:CP_Radial_D7.5mm_P2.50mm, F.Cu at (151.1, 100.3)
- added U8: ADS1115IDGS, Package_SO:TSSOP-10_3x3mm_P0.5mm, F.Cu at (24.1, 55.9)
Connections:
- A1 pad 8: (no net) -> +9V
- A2 pad 8: (no net) -> +9V
- A3 pad 8: (no net) -> +9V
- U1 pad 1: Net-(U1-Pad1) -> (no net)
- U1 pad 27: (no net) -> Net-(U1-Pad27)
- U1 pad 28: (no net) -> Net-(U1-Pad28)
- U7 pad 15: Net-(U1-Pad1) -> Net-(U1-Pad28)
- U7 pad 16: (no net) -> Net-(U1-Pad27)
