File: Aqua.sch (KiCad schematic (older format))
At the start: 21 parts, among them J1 Screw_Terminal_01x02, J2 Screw_Terminal_01x02, J3 Screw_Terminal_01x02, J4 Screw_Terminal_01x02, J5 Screw_Terminal_01x02, J6 Screw_Terminal_01x02, J7 USB_B_Micro, U1 NodeMCU_1.0_(ESP-12E), U2 74HC595, U3 74HC595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

Commit message: WIP
Parts:
- added U8: ADS1115IDGS, Package_SO:TSSOP-10_3x3mm_P0.5mm, symbol Analog_ADC:ADS1115IDGS
- C1, C2, C3: renamed from C?; value CP -> 0.1mF; footprint (none) -> Capacitor_THT:CP_Radial_D7.5mm_P2.50mm
Connections:
- net labels added: +9V
- wire segments 145 -> 178
Other:
- moved on the sheet: C1, C2, C3
Changed lines of the file:
@@
 	13650 2750 13800 2750
 Wire Wire Line
-	13800 2750 13800 2500
+	13800 2750 13800 2650
 Connection ~ 13800 2500
 Wire Wire Line
@@
 	11250 2800 11550 2800
 Wire Wire Line
-	11550 2800 11550 2500
+	11550 2800 11550 2650
 Connection ~ 11550 2500
 Wire Wire Line
@@
 	9500 2850 9700 2850
 Wire Wire Line
-	9700 2850 9700 2500
+	9700 2850 9700 2550
 Connection ~ 9700 2500
 Text GLabel 5100 5350 0    50   Input ~ 0
@@
 Connection ~ 14550 5750
 $Comp
-L power:+3.3V #PWR?
+L power:+3.3V #PWR0108
 U 1 1 5EC8BF19
 P 5250 3800
-F 0 "#PWR?" H 5250 3650 50  0001 C CNN
+F 0 "#PWR0108" H 5250 3650 50  0001 C CNN
 F 1 "+3.3V" H 5265 3973 50  0000 C CNN
 F 2 "" H 5250 3800 50  0001 C CNN
@@
 	5300 3800 5250 3800
 Wire Wire Line
-	3150 1850 2000 1850
-Wire Wire Line
-	2000 1850 2000 4750
-Wire Wire Line
-	2000 4750 4900 4750
-Wire Wire Line
 	8200 1450 8650 1450
 Wire Wire Line
@@
 Wire Wire Line
 	8350 1850 8200 1850
+$Comp
+L Device:CP C2
+U 1 1 5EBB52D4
+P 12050 2500
+F 0 "C2" H 12168 2546 50  0000 L CNN
+F 1 "0.1mF" H 12168 2455 50  0000 L CNN
+F 2 "Capacitor_THT:CP_Radial_D7.5mm_P2.50mm" H 12088 2350 50  0001 C CNN
+F 3 "~" H 12050 2500 50  0001 C CNN
+	1    12050 2500
+	1    0    0    -1
+$EndComp
+$Comp
+L Device:CP C3
+U 1 1 5EBB5A5B
+P 14350 2500
+F 0 "C3" H 14468 2546 50  0000 L CNN
+F 1 "0.1mF" H 14468 2455 50  0000 L CNN
+F 2 "Capacitor_THT:CP_Radial_D7.5mm_P2.50mm" H 14388 2350 50  0001 C CNN
+F 3 "~" H 14350 2500 50  0001 C CNN
+	1    14350 2500
+	1    0    0    -1
+$EndComp
+$Comp
+L Device:CP C1
+U 1 1 5EBB61D6
+P 10200 2300
+F 0 "C1" H 10318 2346 50  0000 L CNN
+F 1 "0.1mF" H 10318 2255 50  0000 L CNN
+F 2 "Capacitor_THT:CP_Radial_D7.5mm_P2.50mm" H 10238 2150 50  0001 C CNN
+F 3 "~" H 10200 2300 50  0001 C CNN
+	1    10200 2300
+	1    0    0    -1
+$EndComp
+$Comp
+L Analog_ADC:ADS1115IDGS U8
+U 1 1 5EBB7CF3
+P 1600 2150
+F 0 "U8" H 1600 2831 50  0000 C CNN
+F 1 "ADS1115IDGS" H 1600 2740 50  0000 C CNN
+F 2 "Package_SO:TSSOP-10_3x3mm_P0.5mm" H 1600 1650 50  0001 C CNN
+F 3 "http://www.ti.com/lit/ds/symlink/ads1113.pdf" H 1550 1250 50  0001 C CNN
+	1    1600 2150
+	1    0    0    -1
+$EndComp
+Text GLabel 1350 2850 0    50   Input ~ 0
+GND
+Wire Wire Line
+	1600 2550 1600 2850
+Wire Wire Line
+	1600 2850 1350 2850
+Wire Wire Line
+	4750 2050 5300 2050
+Wire Wire Line
+	5300 2050 5300 1850
+Wire Wire Line
+	5300 1850 6050 1850
+Wire Wire Line
+	6050 1850 6050 4400
+Wire Wire Line
+	6050 4400 4600 4400
+Wire Wire Line
+	4600 4400 4600 4750
+Wire Wire Line
+	4600 4750 4900 4750
+Wire Wire Line
+	6300 2150 6300 4200
+Wire Wire Line
+	6300 4200 4750 4200
+Wire Wire Line
+	4750 4200 4750 4650
+Wire Wire Line
+	4750 4650 4900 4650
+Wire Wire Line
+	4750 2150 6300 2150
+Wire Wire Line
+	13700 1100 14350 1100
+Wire Wire Line
+	14350 1100 14350 2350
+Wire Wire Line
+	14350 2650 13800 2650
+Connection ~ 13800 2650
+Wire Wire Line
+	13800 2650 13800 2500
+Wire Wire Line
+	12050 2650 11550 2650
+Connection ~ 11550 2650
+Wire Wire Line
+	11550 2650 11550 2500
+Wire Wire Line
+	12050 2350 12050 1000
+Wire Wire Line
+	12050 1000 11450 1000
+Wire Wire Line
+	11450 1000 11450 1100
+Wire Wire Line
+	10200 2150 10700 2150
+Wire Wire Line
+	10700 2150 10700 1050
+Wire Wire Line
+	10700 1050 9600 1050
+Wire Wire Line
+	9600 1050 9600 1100
+Wire Wire Line
+	10200 2450 10200 2550
+Wire Wire Line
+	10200 2550 9700 2550
+Wire Wire Line
+	9700 2550 9700 2500
+Connection ~ 9700 2550
+$Comp
+L power:+9V #PWR0109
+U 1 1 5EC41235
+P 11750 750
+F 0 "#PWR0109" H 11750 600 50  0001 C CNN
+F 1 "+9V" H 11765 923 50  0000 C CNN
+F 2 "" H 11750 750 50  0001 C CNN
+F 3 "" H 11750 750 50  0001 C CNN
+	1    11750 750
+	1    0    0    -1
+$EndComp
+Wire Wire Line
+	10700 1050 10700 750
+Wire Wire Line
+	10700 750  11750 750
+Connection ~ 10700 1050
+Wire Wire Line
+	12050 1000 12050 750
+Wire Wire Line
+	12050 750  11750 750
+Connection ~ 12050 1000
+Connection ~ 11750 750
+Wire Wire Line
+	14350 1100 14350 750
+Wire Wire Line
+	14350 750  12050 750
 Wire Bus Line
 	6500 1050 7300 1050
 Wire Bus Line
 	6450 1250 7300 1250
-$Comp
-L Device:CP C?
-U 1 1 5EBB52D4
-P 6700 5050
-F 0 "C?" H 6818 5096 50  0000 L CNN
-F 1 "CP" H 6818 5005 50  0000 L CNN
-F 2 "" H 6738 4900 50  0001 C CNN
-F 3 "~" H 6700 5050 50  0001 C CNN
-	1    6700 5050
-	1    0    0    -1
-$EndComp
-$Comp
-L Device:CP C?
-U 1 1 5EBB5A5B
-P 7250 5050
-F 0 "C?" H 7368 5096 50  0000 L CNN
-F 1 "CP" H 7368 5005 50  0000 L CNN
-F 2 "" H 7288 4900 50  0001 C CNN
-F 3 "~" H 7250 5050 50  0001 C CNN
-	1    7250 5050
-	1    0    0    -1
-$EndComp
-$Comp
-L Device:CP C?
-U 1 1 5EBB61D6
-P 7850 5050
-F 0 "C?" H 7968 5096 50  0000 L CNN
-F 1 "CP" H 7968 5005 50  0000 L CNN
-F 2 "" H 7888 4900 50  0001 C CNN
-F 3 "~" H 7850 5050 50  0001 C CNN
-	1    7850 5050
-	1    0    0    -1
-$EndComp
+Connection ~ 14350 1100
+Connection ~ 12050 750
 $EndSCHEMATC
